Commit message: Add the simulation loop at the end of the file

File: test.urdf (robot description, URDF)
Before this commit: robot pepe, 5 links, 4 joints
Links:
- added link 25, mass 2.421408511640118; collision cylinder length=1.0594499121012704 radius=0.8529407846695329; visual cylinder length=1.0594499121012704 radius=0.8529407846695329
- link 0: mass 0.08882193011447076 -> 0.19781387757937377; geometry collision cylinder length=0.21925054804629962 radius=0.5358991866661625; visual cylinder length=0.21925054804629962 radius=0.5358991866661625
- link 11: mass 1.3629571017358157 -> 0.1619075375987906; geometry collision cylinder length=0.06835097439446747 radius=0.8683328725871271; visual cylinder length=0.06835097439446747 radius=0.8683328725871271
- link 12: mass 1.3629571017358157 -> 0.1619075375987906; geometry collision cylinder length=0.06835097439446747 radius=0.8683328725871271; visual cylinder length=0.06835097439446747 radius=0.8683328725871271
- link 13: mass 1.3629571017358157 -> 0.1619075375987906; geometry collision cylinder length=0.06835097439446747 radius=0.8683328725871271; visual cylinder length=0.06835097439446747 radius=0.8683328725871271
- link 24: mass 0.00927975494390793 -> 2.421408511640118; geometry collision cylinder length=1.0594499121012704 radius=0.8529407846695329; visual cylinder length=1.0594499121012704 radius=0.8529407846695329
Joints:
- added joint 25_to_0: type revolute, parent 0, child 25, origin xyz=0.48869769270458674 0.1638181490850279 0.8369005404645151 rpy=19.07998851194224 2.7651786030218855 0.3007385672868071, axis 0 1 0, limit lower=3.1415 upper=-3.1415 effort=1 velocity=1
- joint 11_to_0: origin xyz=0.13758607675745194 0.9350807390271525 0.7734982986138889 rpy=1.1448832225386056 4.335027266637536 1.6623373384868418 -> xyz=0.7958007647050853 0.25340169588742434 0.8264867347567081 rpy=8.071640758654594 4.524514626529704 3.066134114242652
- joint 12_to_0: origin xyz=0.13758607675745194 0.9350807390271525 0.7734982986138889 rpy=1.7173248338079086 4.335027266637536 1.6623373384868418 -> xyz=0.7958007647050853 0.25340169588742434 0.8264867347567081 rpy=12.10746113798189 4.524514626529704 3.066134114242652
- joint 13_to_0: origin xyz=0.13758607675745194 0.9350807390271525 0.7734982986138889 rpy=2.2897664450772113 4.335027266637536 1.6623373384868418 -> xyz=0.7958007647050853 0.25340169588742434 0.8264867347567081 rpy=16.143281517309187 4.524514626529704 3.066134114242652
- joint 24_to_0: axis 1 0 0 -> 0 1 0; origin xyz=0.5036286873801603 0.5240689361666607 0.6894713309286168 rpy=25.564766096902733 2.031682406199534 3.494432979573068 -> xyz=0.48869769270458674 0.1638181490850279 0.8369005404645151 rpy=15.899990426618533 2.7651786030218855 0.3007385672868071
